File: Corridor/Corridor.kicad_pcb (KiCad board)
At the start: 2 copper layers, 69.5 x 46.5 mm, 31 parts, among them IC2 SHT31-DIS-B2.5KS, J1 WJ127-5.0-2P, J3 Servo2, J4 RFID, J6 Scale, J7 IR_LEDs, J8 Corridor1, J9 Servo1, Q1 IRLML2502PBF, U1 ADS1114IDGS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

Commit message: Adding fuseholder to the HAT
Parts:
- moved Q1 2.55 mm to (105.0, 81.5)
- moved R9 1.56 mm to (110.5, 81.0)
Routing:
- net +VDC: track 174.8 -> 191.6 mm
- net Net-(Q1-D): track 7.66 -> 10.2 mm
- net Net-(Q1-G): track 4.83 -> 5.42 mm
- net GND: vias 14 -> 19
Other:
- board text added: "+ -"
- board text added: "- + S"
- board text added: "Corridor"
- board text added: "LED"
- board text added: "Servo 1"
- board text added: "Servo 2"
- board text removed: "Corridor 1"
Changed lines of the file:
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@@
 	(footprint "IRLML2502PBF:SOT95P237X112-3N"
 		(layer "F.Cu")
-		(at 104.95 84)
+		(at 104.95 81.45)
 		(descr "SOT-23-ren9")
 		(tags "MOSFET (N-Channel)")
 		(property "Reference" "Q1"
-			(at 0 0 0)
+			(at -3.5 0.05 0)
 			(layer "F.SilkS")
 			(effects
@@
 		(tags "AP2210N-3.3TRG1 ")
 		(property "Reference" "U2"
-			(at 0 0 90)
+			(at 2.55 -0.3375 0)
 			(unlocked yes)
 			(layer "F.SilkS")
@@
 	(footprint "Resistor_SMD:R_1206_3216Metric"
 		(layer "F.Cu")
-		(at 109.9625 82.5 180)
+		(at 110.55 81.05 180)
 		(descr "Resistor SMD 1206 (3216 Metric), square (rectangular) end terminal, IPC-7351 nominal, (Body size source: IPC-SM-782 page 72, https://www.pcb-3d.com/wordpress/wp-content/uploads/ipc-sm-782a_amendment_1_and_2.pdf), generated with kicad-footprint-generator")
 		(tags "resistor")
@@
 		(tags "Integrated Circuit")
 		(property "Reference" "IC2"
-			(at 0 0 90)
+			(at 0.45 -3.85 180)
 			(layer "F.SilkS")
 			(effects
@@
 		(layer "Edge.Cuts")
 	)
+	(gr_text "LED"
+		(at 95.15 85.6 0)
+		(layer "F.SilkS")
+		(effects
+			(font
+				(size 1 1)
+				(thickness 0.1)
+			)
+			(justify left bottom)
+		)
+	)
+	(gr_text "+     -"
+		(at 99.35 85.95 0)
+		(layer "F.SilkS")
+		(effects
+			(font
+				(size 1 1)
+				(thickness 0.1)
+			)
+			(justify left bottom)
+		)
+	)
 	(gr_text "RFID"
 		(at 106.8 51.6 0)
@@
 		)
 	)
+	(gr_text "-  +  S"
+		(at 113.15 91.5 0)
+		(layer "F.SilkS")
+		(effects
+			(font
+				(size 1 1)
+				(thickness 0.1)
+			)
+			(justify left bottom)
+		)
+	)
 	(gr_text "- S+ S- +"
 		(at 113.5 51.2 0)
@@
 		)
 	)
+	(gr_text "Servo 1"
+		(at 113.7 89.85 0)
+		(layer "F.SilkS")
+		(effects
+			(font
+				(size 1 1)
+				(thickness 0.1)
+			)
+			(justify left bottom)
+		)
+	)
 	(gr_text "SCALE"
 		(at 124.8 51.6 0)
@@
 		)
 	)
+	(gr_text "-  +  S"
+		(at 126.1 91.45 0)
+		(layer "F.SilkS")
+		(effects
+			(font
+				(size 1 1)
+				(thickness 0.1)
+			)
+			(justify left bottom)
+		)
+	)
+	(gr_text "Servo 2"
+		(at 126.55 89.65 0)
+		(layer "F.SilkS")
+		(effects
+			(font
+				(size 1 1)
+				(thickness 0.1)
+			)
+			(justify left bottom)
+		)
+	)
 	(gr_text "SHT31"
 		(at 133 55 0)
@@
 		)
 	)
-	(gr_text "Corridor 1"
-		(at 97.6 59.3 270)
+	(gr_text "Corridor"
+		(at 97.7 58.05 270)
 		(layer "F.SilkS")
 		(effects
@@
 	)
 	(segment
-		(start 119.9 80.75)
-		(end 119.224568 80.75)
-		(width 0.2)
-		(layer "F.Cu")
-		(net 1)
-	)
-	(segment
 		(start 129.54 93.5)
 		(end 131.54 95.5)
@@
 	)
 	(segment
-		(start 130 83.5)
-		(end 129.5 84)
-		(width 0.3)
+		(start 118.9 81)
+		(end 118.9 82.3125)
+		(width 0.2)
 		(layer "F.Cu")
 		(net 1)
 	)
 	(segment
-		(start 118.975 82.000432)
-		(end 119.974568 83)
-		(width 0.2)
+		(start 130 83.5)
+		(end 129.5 84)
+		(width 0.3)
 		(layer "F.Cu")
 		(net 1)
@@
 	)
 	(segment
+		(start 129.5 84)
+		(end 137 84)
+		(width 0.3)
+		(layer "F.Cu")
+		(net 1)
+	)
+	(segment
 		(start 143.5 70.5)
 		(end 146.5 67.5)
@@
 	)
 	(segment
+		(start 137 84)
+		(end 143.5 90.5)
+		(width 0.3)
+		(layer "F.Cu")
+		(net 1)
+	)
+	(segment
 		(start 129.262501 81)
 		(end 128.9125 80.649999)
@@
 	)
 	(segment
-		(start 119.224568 80.75)
-		(end 118.975 80.999568)
-		(width 0.2)
-		(layer "F.Cu")
-		(net 1)
-	)
-	(segment
 		(start 128.9125 81.360832)
 		(end 129.273332 81)
@@
 	)
 	(segment
-		(start 121.5 84.9125)
-		(end 119.974568 83.387068)
+		(start 119.15 80.75)
+		(end 118.9 81)
 		(width 0.2)
 		(layer "F.Cu")
@@
 	)
 	(segment
-		(start 119.974568 83.387068)
-		(end 119.974568 83)
-		(width 0.2)
-		(layer "F.Cu")
-		(net 1)
-	)
-	(segment
 		(start 119.9 80.75)
 		(end 119.9 80.25)
@@
 	)
 	(segment
-		(start 118.975 80.999568)
-		(end 118.975 82.000432)
-		(width 0.2)
-		(layer "F.Cu")
-		(net 1)
-	)
-	(segment
 		(start 97.9375 71.9375)
 		(end 100.1812 71.9375)
@@
 	)
 	(segment
+		(start 118.9 82.3125)
+		(end 121.5 84.9125)
+		(width 0.2)
+		(layer "F.Cu")
+		(net 1)
+	)
+	(segment
+		(start 119.9 80.75)
+		(end 119.15 80.75)
+		(width 0.2)
+		(layer "F.Cu")
+		(net 1)
+	)
+	(segment
 		(start 124 83.5)
 		(end 124 82.575)
@@
 	)
 	(via
+		(at 130.85 58.2)
+		(size 0.7)
+		(drill 0.3)
+		(layers "F.Cu" "B.Cu")
+		(free yes)
+		(net 2)
+	)
+	(via
+		(at 131.45 58.75)
+		(size 0.7)
+		(drill 0.3)
+		(layers "F.Cu" "B.Cu")
+		(free yes)
+		(net 2)
+	)
+	(via
 		(at 124.9 56.1)
 		(size 0.7)
@@
 	)
 	(via
+		(at 126.05 79.85)
+		(size 0.7)
+		(drill 0.3)
+		(layers "F.Cu" "B.Cu")
+		(free yes)
+		(net 2)
+	)
+	(via
 		(at 125.7 57)
 		(size 0.7)
@@
 	)
 	(via
+		(at 131.25 59.65)
+		(size 0.7)
+		(drill 0.3)
+		(layers "F.Cu" "B.Cu")
+		(free yes)
+		(net 2)
+	)
+	(via
 		(at 100 75)
 		(size 0.7)
@@
 		(net 2)
 	)
+	(via
+		(at 125.95 78.85)
+		(size 0.7)
+		(drill 0.3)
+		(layers "F.Cu" "B.Cu")
+		(free yes)
+		(net 2)
+	)
 	(segment
 		(start 118 69.5)
@@
 	)
 	(segment
-		(start 106 84)
+		(start 105.25 91.35)
 		(end 106 90.6)
 		(width 0.7)
@@
 	(segment
 		(start 106 90.6)
-		(end 105.25 91.35)
+		(end 106 81.45)
 		(width 0.7)
 		(layer "F.Cu")
@@
 	)
 	(segment
-		(start 118.025 81.000432)
-		(end 118.025 74.525)
+		(start 118.15 74.65)
+		(end 118 74.5)
+		(width 0.2)
+		(layer "F.Cu")
+		(net 10)
+	)
+	(segment
+		(start 118.15 74.703553)
+		(end 118.15 74.65)
 		(width 0.2)
 		(layer "F.Cu")
@@
 	)
 	(segment
+		(start 117.1 81.25)
+		(end 117.94703 81.25)
+		(width 0.2)
+		(layer "F.Cu")
+		(net 10)
+	)
+	(segment
 		(start 121 70.713348)
 		(end 120.5 71.213348)
@@
 	)
 	(segment
-		(start 117.1 81.25)
-		(end 117.775432 81.25)
+		(start 117.94703 81.25)
+		(end 118.1 81.09703)
 		(width 0.2)
 		(layer "F.Cu")
@@
 	)
 	(segment
-		(start 118.025 74.525)
-		(end 118 74.5)
+		(start 118.1 81.09703)
+		(end 118.1 74.753553)
 		(width 0.2)
 		(layer "F.Cu")
@@
 	)
 	(segment
-		(start 117.775432 81.25)
-		(end 118.025 81.000432)
+		(start 118.1 74.753553)
+		(end 118.15 74.703553)
 		(width 0.2)
 		(layer "F.Cu")
@@
 	)
 	(segment
-		(start 104.45 82.5)
-		(end 103.9 83.05)
+		(start 103.9 80.5)
+		(end 108.5375 80.5)
 		(width 0.3)
 		(layer "F.Cu")
@@
 	)
 	(segment
-		(start 108.5 82.5)
-		(end 104.45 82.5)
+		(start 108.5375 80.5)
+		(end 109.0875 81.05)
 		(width 0.3)
 		(layer "F.Cu")
@@
 	)
 	(segment
-		(start 116.425 87.5)
-		(end 111.425 82.5)
+		(start 112.0125 81.0625)
+		(end 112.0125 81.05)
 		(width 0.3)
 		(layer "F.Cu")
@@
 	)
 	(segment
-		(start 124.25 87.5)
-		(end 116.425 87.5)
+		(start 130 75.15)
+		(end 129.148289 75.15)
 		(width 0.3)
 		(layer "F.Cu")
@@
 	)
 	(segment
-		(start 130 75.15)
-		(end 129.148289 75.15)
+		(start 118.45 87.5)
+		(end 112.0125 81.0625)
 		(width 0.3)
 		(layer "F.Cu")
@@
 	)
 	(segment
-		(start 127.4125 76.885789)
-		(end 127.4125 84.3375)
+		(start 127.4125 84.3375)
+		(end 124.25 87.5)
 		(width 0.3)
 		(layer "F.Cu")
@@
 	)
 	(segment
-		(start 127.4125 84.3375)
-		(end 124.25 87.5)
+		(start 124.25 87.5)
+		(end 118.45 87.5)
+		(width 0.3)
+		(layer "F.Cu")
+		(net 32)
+	)
+	(segment
+		(start 127.4125 76.885789)
+		(end 127.4125 84.3375)
 		(width 0.3)
 		(layer "F.Cu")
