File: Corridor/Corridor.kicad_pcb (KiCad board)
At the start: 2 copper layers, 69.5 x 46.5 mm, 31 parts, among them IC2 SHT31-DIS-B2.5KS, J1 WJ127-5.0-2P, J3 Servo2, J4 RFID, J6 Scale, J7 IR_LEDs, J8 Corridor1, J9 Servo1, Q1 IRLML2502PBF, U1 ADS1114IDGS, U2 AP2210N-3.3TRG1, U3 AD8293G80ARJZ-R7, U4 PCA9685PW, U5 PCA9306

Commit message: v1.0
Parts:
- added J10: FC68148, FC68148:FC68148, F.Cu at (96.0, 75.1)
- added J2: Servo3, Connector_PinHeader_2.54mm:PinHeader_1x03_P2.54mm_Vertical, F.Cu at (108.5, 93.5)
- added J5: Servo4, Connector_PinHeader_2.54mm:PinHeader_1x03_P2.54mm_Vertical, F.Cu at (98.0, 93.5)
- moved J1 14.0 mm to (86.2, 90.8)
- moved J3 5.00 mm to (118.9, 93.5)
- moved C2 4.22 mm to (101.5, 75.7)
- moved U2 4.22 mm to (105.0, 74.2)
- moved C4 3.83 mm to (111.2, 73.1)
- moved J9 1.92 mm to (128.9, 93.5)
Connections:
- J8 pad 8: +VDC -> unconnected-(J8-Pad8)
- R9 pad 1: STRIP_PWM -> Net-(U4-LED8)
- U4 pad 12: STRIP_PWM -> Net-(J2-Pin_3)
- U4 pad 13: unconnected-(U4-LED7-Pad13) -> Net-(J5-Pin_3)
- U4 pad 15: unconnected-(U4-LED8-Pad15) -> Net-(U4-LED8)
Routing:
- net Net-(J5-Pin_3): track 0.00 -> 39.2 mm
- net STRIP_PWM: track 30.1 -> 0.00 mm
- net Net-(J2-Pin_3): track 0.00 -> 28.4 mm
- net Net-(U4-LED8): track 0.00 -> 21.2 mm, vias 0 -> 2
- net Net-(Q1-D): track 10.2 -> 19.6 mm
- net +VDC: track 191.6 -> 185.2 mm
- net Net-(J3-Pin_3): track 24.8 -> 20.7 mm
- net +3.3VA: track 98.1 -> 96.1 mm
- net Net-(J9-Pin_3): track 19.7 -> 20.5 mm
Other:
- board text added: "Servo 3"
- board text added: "Servo 4"
- board text removed: "Corridor"
