File: RPiShield/RPiShield.kicad_pcb (KiCad board)
At the start: 2 copper layers, 65 x 56.5 mm, 6 parts, among them J2 BBOX, J4 Corridor1, J7 FC68148, J8 2223

Commit message: v1.0
Parts:
- added J1: FC68148, FC68148:FC68148, F.Cu at (179.8, 56.6)
- added J3: FC68148, FC68148:FC68148, F.Cu at (158.0, 81.6)
- moved J2 10.9 mm to (193.4, 88.8)
- moved F1 4.65 mm to (164.7, 55.0)
- moved F2 4.45 mm to (164.7, 70.0)
- moved J4 2.29 mm to (157.6, 96.5)
Connections:
- J2 pad 8: Net-(F1-Pad1) -> SWITCH
- J4 pad 8: Net-(F2-Pad1) -> unconnected-(J4-Pad8)
- J8 pad 38: unconnected-(J8-Pad38) -> SWITCH
Routing:
- net SWITCH: track 0.00 -> 26.5 mm
- net I2C_SCL: track 83.7 -> 74.0 mm
- net LED: track 31.9 -> 40.7 mm
- net I2C_SDA: track 88.9 -> 81.0 mm
- net Net-(F2-Pad1): track 23.3 -> 16.0 mm
- net Net-(F1-Pad1): track 19.1 -> 15.9 mm
- net RFID_TX: track 77.9 -> 76.4 mm
- net GND: track 0.00 -> 0.68 mm
Other:
- board size 65 x 56.5 mm -> 65.6 x 56.5 mm
- board text added: "+5V"
- board text added: "Box"
- board text removed: "BBOX"
